File: MouseProject/mouse/mouse.kicad_sch (KiCad schematic)
At the start: 66 parts, among them J1 B4B-PH-K-S_LF__SN_, J2 B02B-PASK-1, J3 B4B-PH-K-S_LF__SN_, J4 5051100492, J5 USB_B_Micro, J6 5051100492, Q7 MMBT3904-7-F, Q8 MMBT3904-7-F, Q9 MMBT3904-7-F, U1 AP2112K-3.3, U2 MIC5219-5.0YM5-TR, U3 TPS78319DDCT

Commit message: Update for final board rev1
Parts:
- removed C15: 22uF, Capacitor_SMD:C_0201_0603Metric, symbol c_small:C_Small
- removed C16: 0.1uF, Capacitor_SMD:C_0201_0603Metric, symbol c_small:C_Small
- removed C18, C19, C20: 4.7uF, Capacitor_SMD:C_0201_0603Metric, symbol c_small:C_Small
- removed D6: LED_R, LED_SMD:LED_0201_0603Metric, symbol LED_small:LED
- removed D7: LED_G, LED_SMD:LED_0201_0603Metric, symbol LED_small:LED
- removed D8: LED_B, LED_SMD:LED_0201_0603Metric, symbol LED_small:LED
- removed J1, J3: B4B-PH-K-S_LF__SN_, digikey-footprints:PinHeader_1x4_P2mm_Drill1mm, symbol conn_4pin_2mm:B4B-PH-K-S_LF__SN_
- removed Q7, Q8, Q9: MMBT3904-7-F, digikey-footprints:SOT-23-3, symbol dk_Transistors-Bipolar-BJT-Single:MMBT3904-7-F
- removed R22, R23, R24: ??, Resistor_SMD:R_0201_0603Metric, symbol r_small:R_Small
- removed U2: MIC5219-5.0YM5-TR, MIC5219_5_0YM5_TR:SOT-23-5_M5_MCH, symbol ap2112k_3v3:AP2112K-3.3
- added R12, R13, R14, R19, R20: 10k, Resistor_SMD:R_0201_0603Metric, symbol r_small:R_Small
Connections:
- net PWR_5V_EN is gone; now on net SW4_COM: ESP1.18 (IO10)
- net +3.3V: now also R12.1, R13.1, R14.1, R19.1, R20.1; no longer LMB1.2 (NO), MMB1.2 (NO), RMB1.2 (NO)
- net -BATT: now also LMB1.1 (COM), RMB1.1 (COM); no longer LMB1.3 (NC), RMB1.3 (NC)
- net PWR_EN: no longer U3.3 (EN)
- net SW3_COM: now also ESP1.19 (IO11), J6.3; no longer ESP1.6 (IO6), J6.1
- net SW3_COM_OFF: now also J4.4; no longer J4.1
- net SW4_COM: now also J6.4; no longer ESP1.7 (IO7), J6.2
- net SW4_COM_OFF: now also J4.3; no longer J4.2
- net PWR_1.9V_EN: now reaches ESP1.39 (IO1)
- net PWR_1.9V_EN: now also U3.3 (EN)
- net SW1_COM renamed SW1_NO
- net SW1_NO: now also LMB1.2 (NO), R14.2; no longer LMB1.1 (COM)
- net SW2_COM renamed SW1_NC
- net SW1_NC: now also LMB1.3 (NC), R13.2; no longer RMB1.1 (COM)
- new net SW2_NC: ESP1.7 (IO7), R19.2, RMB1.3 (NC)
- new net SW2_NO: ESP1.6 (IO6), R20.2, RMB1.2 (NO)
- new net SW5_NO: MMB1.2 (NO), R12.2
Other:
- moved on the sheet: J4, J6
